Commit message: 新增gazebo仿真，用于底盘仿真；urdf增加gazebo依赖；关闭gazebo动力学仿真，仅支持运动学仿真；

File: src/mantis_description/urdf/mantis copy.urdf (robot description, URDF)
Before this commit: robot mantis, 28 links, 27 joints
Joints:
- joint Head_Joint: limit lower=-0.7 upper=0.2 effort=1000 velocity=10 -> lower=-0.7 upper=0.2 effort=0 velocity=0
- joint L_Ear_Joint: limit lower=-1.57 upper=0.5 effort=1000 velocity=10 -> lower=-1.57 upper=0.5 effort=0 velocity=0
- joint L_Elbow_Pitch_Joint: limit lower=-0.395 upper=1.012 effort=1000 velocity=10 -> lower=-0.395 upper=1.012 effort=0 velocity=0
- joint L_Hand_L_Joint: limit lower=0.0 upper=0.04 effort=1000 velocity=10 -> lower=0.0 upper=0.04 effort=0 velocity=0
- joint L_Hand_R_Joint: limit lower=0.0 upper=0.04 effort=1000 velocity=10 -> lower=0.0 upper=0.04 effort=0 velocity=0
- joint L_Shoulder_Pitch_Joint: limit lower=-1.13 upper=1.75 effort=1000 velocity=10 -> lower=-1.13 upper=1.75 effort=0 velocity=0
- joint L_Shoulder_Roll_Joint: limit lower=-0.8 upper=0.82 effort=1000 velocity=10 -> lower=-0.8 upper=0.82 effort=0 velocity=0
- joint L_Shoulder_Yaw_Joint: limit lower=-0.213 upper=2.029 effort=1000 velocity=10 -> lower=-0.213 upper=2.029 effort=0 velocity=0
- joint L_Wrist_Pitch_Joint: limit lower=-0.562 upper=0.562 effort=1000 velocity=10 -> lower=-0.562 upper=0.562 effort=0 velocity=0
- joint L_Wrist_Roll_Joint: limit lower=-1.7 upper=1.7 effort=1000 velocity=10 -> lower=-1.7 upper=1.7 effort=0 velocity=0
- joint L_Wrist_Yaw_Joint: limit lower=-1.7 upper=1.7 effort=1000 velocity=10 -> lower=-1.7 upper=1.7 effort=0 velocity=0
- joint Neck_Joint: limit lower=-1.57 upper=1.57 effort=1000 velocity=10 -> lower=-1.57 upper=1.57 effort=0 velocity=0
- joint R_Ear_Joint: limit lower=-1.57 upper=0.5 effort=1000 velocity=10 -> lower=-1.57 upper=0.5 effort=0 velocity=0
- joint R_Elbow_Pitch_Joint: limit lower=-0.395 upper=1.012 effort=1000 velocity=10 -> lower=-0.395 upper=1.012 effort=0 velocity=0
- joint R_Hand_L_Joint: limit lower=0.0 upper=0.04 effort=1000 velocity=10 -> lower=0.0 upper=0.04 effort=0 velocity=0
- joint R_Hand_R_Joint: limit lower=0.0 upper=0.04 effort=1000 velocity=10 -> lower=0.0 upper=0.04 effort=0 velocity=0
- joint R_Shoulder_Pitch_Joint: limit lower=-1.13 upper=1.75 effort=1000 velocity=10 -> lower=-1.13 upper=1.75 effort=0 velocity=0
- joint R_Shoulder_Roll_Joint: limit lower=-0.8 upper=0.82 effort=1000 velocity=10 -> lower=-0.8 upper=0.82 effort=0 velocity=0
- joint R_Shoulder_Yaw_Joint: limit lower=-0.213 upper=2.029 effort=1000 velocity=10 -> lower=-0.213 upper=2.029 effort=0 velocity=0
- joint R_Wrist_Pitch_Joint: limit lower=-0.562 upper=0.562 effort=1000 velocity=10 -> lower=-0.562 upper=0.562 effort=0 velocity=0
- joint R_Wrist_Roll_Joint: limit lower=-1.7 upper=1.7 effort=1000 velocity=10 -> lower=-1.7 upper=1.7 effort=0 velocity=0
- joint R_Wrist_Yaw_Joint: limit lower=-1.7 upper=1.7 effort=1000 velocity=10 -> lower=-1.7 upper=1.7 effort=0 velocity=0
- joint Waist_Joint: limit lower=-0.62 upper=0.24 effort=1000 velocity=10 -> lower=-0.62 upper=0.24 effort=0 velocity=0
- joint Wheel_Back_Joint: axis (none) -> 0 0 -1; type fixed -> continuous
- joint Wheel_Left_Joint: axis (none) -> 0 0 -1; type fixed -> continuous
- joint Wheel_Right_Joint: axis (none) -> 0 0 -1; type fixed -> continuous
