Commit message: 优化urdf，增加夹爪模型；

File: src/mantis_description/urdf/mantis.urdf (robot description, URDF)
Before this commit: robot mantis, 28 links, 27 joints
Joints:
- joint L_Elbow_Pitch_Joint: origin xyz=0 -0.0140000000000004 -0.35448 rpy=1.5707963267949 0.147258361384734 3.14159265358979 -> xyz=0 -0.0139999999999995 -0.35448 rpy=1.5707963267949 0.147258361384734 3.14159265358979
- joint R_Elbow_Pitch_Joint: origin xyz=0 -0.0140000000000004 -0.35448 rpy=1.5707963267949 0.147258361384736 3.14159265358979 -> xyz=0 -0.0140000000000004 -0.354479999999999 rpy=1.5707963267949 0.147258361384736 3.14159265358979
- joint R_Shoulder_Yaw_Joint: axis 0 0 1 -> 0 0 -1
- joint R_Wrist_Pitch_Joint: axis 0 0 1 -> 0 0 -1
- joint R_Wrist_Roll_Joint: axis 0 0 1 -> 0 0 -1
- joint R_Wrist_Yaw_Joint: axis 0 -0.0452652870134508 0.998975001584919 -> 0 -0.0452652870134508 -0.998975001584919

Commit message: 增加gui模式夹爪控制；解决关节限位数据错误bug；解决ik模式大面积穿摸bug；

File: src/mantis_description/urdf/mantis.urdf (robot description, URDF)
Before this commit: robot mantis, 28 links, 27 joints
Links:
- link Head_Link: geometry collision mesh filename=package://mantis_description/meshes/collision/Head_Link.STL; visual mesh filename=package://mantis_description/meshes/visual/Head_Link.STL
- link L_Ear_Link: geometry collision mesh filename=package://mantis_description/meshes/collision/L_Ear_Link.STL; visual mesh filename=package://mantis_description/meshes/visual/L_Ear_Link.STL
- link L_Elbow_Pitch_Link: geometry collision mesh filename=package://mantis_description/meshes/collision/L_Elbow_Pitch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; visual mesh filename=package://mantis_description/meshes/visual/L_Elbow_Pitch_Li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
- link L_Hand_L_Link: geometry collision mesh filename=package://mantis_description/meshes/collision/L_Hand_L_Link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; visual mesh filename=package://mantis_description/meshes/visual/L_Hand_L_Link.STL
- link L_Hand_R_Link: geometry collision mesh filename=package://mantis_description/meshes/collision/L_Hand_R_Link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; visual mesh filename=package://mantis_description/meshes/visual/L_Hand_R_Link.STL
- link L_Shoulder_Pitch_Link: geometry collision mesh filename=package://mantis_description/meshes/collision/L_Shoulder_Pi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; visual mesh filename=package://mantis_description/meshes/visual/L_Shoulder_Pitch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
- link L_Shoulder_Roll_Link: geometry collision mesh filename=package://mantis_description/meshes/collision/L_Shoulder_Ro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; visual mesh filename=package://mantis_description/meshes/visual/L_Shoulder_Roll_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
- link L_Shoulder_Yaw_Link: geometry collision mesh filename=package://mantis_description/meshes/collision/L_Shoulder_Ya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; visual mesh filename=package://mantis_description/meshes/visual/L_Shoulder_Yaw_L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
- link L_Wrist_Pitch_Link: geometry collision mesh filename=package://mantis_description/meshes/collision/L_Wrist_Pitch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; visual mesh filename=package://mantis_description/meshes/visual/L_Wrist_Pitch_Li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
- link L_Wrist_Roll_Link: geometry collision mesh filename=package://mantis_description/meshes/collision/L_Wrist_Roll_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; visual mesh filename=package://mantis_description/meshes/visual/L_Wrist_Roll_Lin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
- link L_Wrist_Yaw_Link: geometry collision mesh filename=package://mantis_description/meshes/collision/L_Wrist_Yaw_L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; visual mesh filename=package://mantis_description/meshes/visual/L_Wrist_Yaw_Link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
- link Neck_Link: geometry collision mesh filename=package://mantis_description/meshes/collision/Neck_Link.STL; visual mesh filename=package://mantis_description/meshes/visual/Neck_Link.STL
- link R_Ear_Link: geometry collision mesh filename=package://mantis_description/meshes/collision/R_Ear_Link.STL; visual mesh filename=package://mantis_description/meshes/visual/R_Ear_Link.STL
- link R_Elbow_Pitch_Link: geometry collision mesh filename=package://mantis_description/meshes/collision/R_Elbow_Pitch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; visual mesh filename=package://mantis_description/meshes/visual/R_Elbow_Pitch_Li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
- link R_Hand_L_Link: geometry collision mesh filename=package://mantis_description/meshes/collision/R_Hand_L_Link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; visual mesh filename=package://mantis_description/meshes/visual/R_Hand_L_Link.STL
- link R_Hand_R_Link: geometry collision mesh filename=package://mantis_description/meshes/collision/R_Hand_R_Link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; visual mesh filename=package://mantis_description/meshes/visual/R_Hand_R_Link.STL
- link R_Shoulder_Pitch_Link: geometry collision mesh filename=package://mantis_description/meshes/collision/R_Shoulder_Pi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; visual mesh filename=package://mantis_description/meshes/visual/R_Shoulder_Pitch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
- link R_Shoulder_Roll_Link: geometry collision mesh filename=package://mantis_description/meshes/collision/R_Shoulder_Ro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; visual mesh filename=package://mantis_description/meshes/visual/R_Shoulder_Roll_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
- link R_Shoulder_Yaw_Link: geometry collision mesh filename=package://mantis_description/meshes/collision/R_Shoulder_Ya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; visual mesh filename=package://mantis_description/meshes/visual/R_Shoulder_Yaw_L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
- link R_Wrist_Pitch_Link: geometry collision mesh filename=package://mantis_description/meshes/collision/R_Wrist_Pitch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; visual mesh filename=package://mantis_description/meshes/visual/R_Wrist_Pitch_Li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
- link R_Wrist_Roll_Link: geometry collision mesh filename=package://mantis_description/meshes/collision/R_Wrist_Roll_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; visual mesh filename=package://mantis_description/meshes/visual/R_Wrist_Roll_Lin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
- link R_Wrist_Yaw_Link: geometry collision mesh filename=package://mantis_description/meshes/collision/R_Wrist_Yaw_L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; visual mesh filename=package://mantis_description/meshes/visual/R_Wrist_Yaw_Link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
- link Waist_Link: geometry collision mesh filename=package://mantis_description/meshes/collision/Waist_Link.STL; visual mesh filename=package://mantis_description/meshes/visual/Waist_Link.STL
- link Wheel_Back_Link: geometry collision mesh filename=package://mantis_description/meshes/collision/Wheel_Back_Li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; visual mesh filename=package://mantis_description/meshes/visual/Wheel_Back_Link.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
- link Wheel_Left_Link: geometry collision mesh filename=package://mantis_description/meshes/collision/Wheel_Left_Li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; visual mesh filename=package://mantis_description/meshes/visual/Wheel_Left_Link.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
- link Wheel_Right_Link: geometry collision mesh filename=package://mantis_description/meshes/collision/Wheel_Right_L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; visual mesh filename=package://mantis_description/meshes/visual/Wheel_Right_Link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
- link base_link: geometry collision mesh filename=package://mantis_description/meshes/collision/base_link.STL; visual mesh filename=package://mantis_description/meshes/visual/base_link.STL
Joints:
- joint L_Elbow_Pitch_Joint: limit lower=-0.78 upper=1.57 effort=0 velocity=0 -> lower=-0.395 upper=1.012 effort=0 velocity=0
- joint L_Hand_L_Joint: limit lower=0 upper=0.04 effort=0 velocity=0 -> lower=0.0 upper=0.04 effort=0 velocity=0
- joint L_Hand_R_Joint: limit lower=0 upper=0.04 effort=0 velocity=0 -> lower=0.0 upper=0.04 effort=0 velocity=0
- joint L_Shoulder_Pitch_Joint: limit lower=-2.61 upper=0.78 effort=0 velocity=0 -> lower=-1.13 upper=1.75 effort=0 velocity=0
- joint L_Shoulder_Roll_Joint: limit lower=-1.57 upper=1.57 effort=0 velocity=0 -> lower=-0.8 upper=0.82 effort=0 velocity=0
- joint L_Shoulder_Yaw_Joint: limit lower=0.08 upper=1.04 effort=0 velocity=0 -> lower=-0.213 upper=2.029 effort=0 velocity=0
- joint L_Wrist_Pitch_Joint: limit lower=-0.52 upper=0.52 effort=0 velocity=0 -> lower=-0.562 upper=0.562 effort=0 velocity=0
- joint L_Wrist_Roll_Joint: limit lower=-1.57 upper=1.57 effort=0 velocity=0 -> lower=-1.7 upper=1.7 effort=0 velocity=0
- joint L_Wrist_Yaw_Joint: limit lower=-1.57 upper=1.57 effort=0 velocity=0 -> lower=-1.7 upper=1.7 effort=0 velocity=0
- joint R_Elbow_Pitch_Joint: limit lower=-0.78 upper=1.57 effort=0 velocity=0 -> lower=-0.395 upper=1.012 effort=0 velocity=0
- joint R_Hand_L_Joint: limit lower=0 upper=0.04 effort=0 velocity=0 -> lower=0.0 upper=0.04 effort=0 velocity=0
- joint R_Hand_R_Joint: limit lower=0 upper=0.04 effort=0 velocity=0 -> lower=0.0 upper=0.04 effort=0 velocity=0
- joint R_Shoulder_Pitch_Joint: limit lower=-2.61 upper=0.78 effort=0 velocity=0 -> lower=-1.13 upper=1.75 effort=0 velocity=0
- joint R_Shoulder_Roll_Joint: limit lower=-1.57 upper=1.57 effort=0 velocity=0 -> lower=-0.8 upper=0.82 effort=0 velocity=0
- joint R_Shoulder_Yaw_Joint: limit lower=-1.04 upper=-0.08 effort=0 velocity=0 -> lower=-0.213 upper=2.029 effort=0 velocity=0
- joint R_Wrist_Pitch_Joint: limit lower=-0.52 upper=0.52 effort=0 velocity=0 -> lower=-0.562 upper=0.562 effort=0 velocity=0
- joint R_Wrist_Roll_Joint: limit lower=-1.57 upper=1.57 effort=0 velocity=0 -> lower=-1.7 upper=1.7 effort=0 velocity=0
- joint R_Wrist_Yaw_Joint: limit lower=-1.57 upper=1.57 effort=0 velocity=0 -> lower=-1.7 upper=1.7 effort=0 velocity=0

Commit message: 修复urdf双臂初始位姿不一致的问题；更新readme；

File: src/mantis_description/urdf/mantis.urdf (robot description, URDF)
Before this commit: robot mantis, 28 links, 27 joints
Joints:
- joint R_Elbow_Pitch_Joint: origin xyz=0 -0.0140000000000004 -0.354479999999999 rpy=1.5707963267949 0.147258361384736 3.14159265358979 -> xyz=0 -0.0140000000000004 -0.354479999999999 rpy=1.5707963267949 -0.01000000000 3.14159265358979
- joint R_Shoulder_Pitch_Joint: origin xyz=0.119415661636301 0.133000000337764 0.138469895775482 rpy=1.13289646330337 0.0818475244724988 1.53253534072457 -> xyz=0.119415661636301 0.112951840620579 0.138469895775482 rpy=1.13289646330337 0.0818475244724988 1.53253534072457
- joint R_Shoulder_Yaw_Joint: origin xyz=-0.105087634007942 -0.00931875405517957 0.109999999999979 rpy=1.57079632679489 1.13446263104148 1.65924101328647 -> xyz=-0.0851253117883655 -0.00746534000720467 0.109999999999979 rpy=1.57079632679489 1.13446263104148 1.65924101328647
